File: bkm-68x-video.sch (KiCad schematic (older format))
At the start: 50 parts, among them J1 Y_G, J10 TP_VIDEO_OE, J11 TP_VSYNC, J2 PB_B, J3 PR_R, J4 EXT_SYNC, J5 TP_Y_G, J6 TP_PB_B, J7 TP_PR_R, J8 TP_HSYNC, J9 TP_INT_EXT_SYNC, U1 ADG1611, U2 THS7374, U3 ISL59885, U4 ADG734, U8 TC7WH125

Commit message: A lotta fixes
Parts:
- added R42, R43: R, Resistor_SMD:R_0805_2012Metric_Pad1.20x1.40mm_HandSolder, symbol bkm-68x-simple-rescue:R
- added R71, R72: 47R, Resistor_SMD:R_0805_2012Metric_Pad1.20x1.40mm_HandSolder, symbol bkm-68x-simple-rescue:R
- J1: value Y_G -> PR_R
- J2: value PB_B -> Y_G
- J3: value PR_R -> PB_B
- U4: footprint Package_SO:TSSOP-16_4.4x5mm_P0.65mm -> Package_SO:TSSOP-20_4.4x6.5mm_P0.65mm
Connections:
- wire segments 90 -> 94
Changed lines of the file:
@@
 Wire Wire Line
 	3650 5800 3800 5800
-Text GLabel 3200 5800 0    60   Input ~ 0
+Text GLabel 2900 5800 0    60   Input ~ 0
 VSYNC_SEP
 Connection ~ 3300 5800
@@
 Connection ~ 5350 6000
 Connection ~ 5450 5600
-Text GLabel 5600 5600 2    60   Input ~ 0
+Text GLabel 5900 5600 2    60   Input ~ 0
 HSYNC_SEP
 $Comp
@@
 P 900 1100
 F 0 "J1" H 910 1220 50  0000 C CNN
-F 1 "Y_G" V 1015 1100 50  0000 C CNN
+F 1 "PR_R" V 1015 1100 50  0000 C CNN
 F 2 "BNC-THT:BNC-THT" H 900 1100 50  0001 C CNN
 F 3 "" H 900 1100 50  0001 C CNN
@@
 	-1   0    0    1
 $EndComp
-Text GLabel 1700 1100 2    60   Input ~ 0
+Text GLabel 1700 2150 2    60   Input ~ 0
 Y_G_IN
 $Comp
@@
 P 900 3200
 F 0 "J3" H 910 3320 50  0000 C CNN
-F 1 "PR_R" V 1015 3200 50  0000 C CNN
+F 1 "PB_B" V 1015 3200 50  0000 C CNN
 F 2 "BNC-THT:BNC-THT" H 900 3200 50  0001 C CNN
 F 3 "" H 900 3200 50  0001 C CNN
@@
 	-1   0    0    1
 $EndComp
-Text GLabel 1700 3200 2    60   Input ~ 0
+Text GLabel 1700 1100 2    60   Input ~ 0
 PR_R_IN
 $Comp
@@
 P 900 2150
 F 0 "J2" H 910 2270 50  0000 C CNN
-F 1 "PB_B" V 1015 2150 50  0000 C CNN
+F 1 "Y_G" V 1015 2150 50  0000 C CNN
 F 2 "BNC-THT:BNC-THT" H 900 2150 50  0001 C CNN
 F 3 "" H 900 2150 50  0001 C CNN
@@
 	-1   0    0    1
 $EndComp
-Text GLabel 1700 2150 2    60   Input ~ 0
+Text GLabel 1700 3200 2    60   Input ~ 0
 PB_B_IN
 $Comp
@@
 Wire Wire Line
 	3600 1850 3700 1850
+Text GLabel 3400 1550 0    60   Input ~ 0
+Y_G_IN
+Text GLabel 3400 1700 0    60   Input ~ 0
+PB_B_IN
 Text GLabel 3400 1400 0    60   Input ~ 0
-Y_G_IN
-Text GLabel 3400 1550 0    60   Input ~ 0
-PB_B_IN
-Text GLabel 3400 1700 0    60   Input ~ 0
 PR_R_IN
 $Comp
@@
 $EndComp
 $Comp
-L power:GNDA #PWR014
-U 1 1 5F26B60D
-P 4900 2200
-F 0 "#PWR014" H 4900 1950 50  0001 C CNN
-F 1 "GNDA" V 4900 2000 50  0000 C CNN
-F 2 "" H 4900 2200 50  0001 C CNN
-F 3 "" H 4900 2200 50  0001 C CNN
-	1    4900 2200
-	0    -1   -1   0
-$EndComp
-$Comp
 L adg734:ADG734 U4
 U 1 1 5F26BA5F
@@
 F 0 "U4" H 4800 3650 60  0000 C CNN
 F 1 "ADG734" H 4200 3650 60  0000 C CNN
-F 2 "Package_SO:TSSOP-16_4.4x5mm_P0.65mm" H 4250 4400 60  0001 C CNN
+F 2 "Package_SO:TSSOP-20_4.4x6.5mm_P0.65mm" H 4250 4400 60  0001 C CNN
 F 3 "" H 4250 4400 60  0001 C CNN
 	1    4400 4100
 	1    0    0    -1
 $EndComp
-Text GLabel 4900 1550 2    60   Input ~ 0
-Y_G_AMP
 Text GLabel 4900 1700 2    60   Input ~ 0
 PB_B_AMP
@@
 $EndComp
 Wire Wire Line
-	4900 2050 5200 2050
+	4900 2050 5000 2050
 Wire Wire Line
 	5300 2250 5200 2250
@@
 Connection ~ 7900 2950
 NoConn ~ 4900 6000
-Text GLabel 9250 4450 2    60   Input ~ 0
+Text GLabel 9550 4450 2    60   Input ~ 0
 HSYNC
 $Comp
@@
 Text GLabel 8550 4450 0    60   Input ~ 0
 HSYNC_OUT
-Text GLabel 9250 5250 2    60   Input ~ 0
+Text GLabel 9550 5250 2    60   Input ~ 0
 VSYNC
 Text GLabel 8550 4200 0    60   Input ~ 0
@@
 	0    -1   -1   0
 $EndComp
+Wire Wire Line
+	4900 2200 5000 2200
+Wire Wire Line
+	5000 2200 5000 2050
+Connection ~ 5000 2050
+Wire Wire Line
+	5000 2050 5200 2050
+Text GLabel 4900 1550 2    60   Input ~ 0
+Y_G_AMP
+$Comp
+L bkm-68x-simple-rescue:R R71
+U 1 1 60729AD2
+P 9400 4450
+F 0 "R71" V 9480 4450 50  0000 C CNN
+F 1 "47R" V 9400 4450 50  0000 C CNN
+F 2 "Resistor_SMD:R_0805_2012Metric_Pad1.20x1.40mm_HandSolder" V 9330 4450 50  0001 C CNN
+F 3 "" H 9400 4450 50  0001 C CNN
+	1    9400 4450
+	0    -1   -1   0
+$EndComp
+$Comp
+L bkm-68x-simple-rescue:R R72
+U 1 1 6072CA13
+P 9400 5250
+F 0 "R72" V 9480 5250 50  0000 C CNN
+F 1 "47R" V 9400 5250 50  0000 C CNN
+F 2 "Resistor_SMD:R_0805_2012Metric_Pad1.20x1.40mm_HandSolder" V 9330 5250 50  0001 C CNN
+F 3 "" H 9400 5250 50  0001 C CNN
+	1    9400 5250
+	0    -1   -1   0
+$EndComp
+$Comp
+L bkm-68x-simple-rescue:R R43
+U 1 1 608268F3
+P 3050 5800
+F 0 "R43" V 3130 5800 50  0000 C CNN
+F 1 "R" V 3050 5800 50  0000 C CNN
+F 2 "Resistor_SMD:R_0805_2012Metric_Pad1.20x1.40mm_HandSolder" V 2980 5800 50  0001 C CNN
+F 3 "" H 3050 5800 50  0001 C CNN
+	1    3050 5800
+	0    -1   -1   0
+$EndComp
+Wire Wire Line
+	2800 5800 2900 5800
+$Comp
+L bkm-68x-simple-rescue:R R42
+U 1 1 60830305
+P 5750 5600
+F 0 "R42" V 5830 5600 50  0000 C CNN
+F 1 "R" V 5750 5600 50  0000 C CNN
+F 2 "Resistor_SMD:R_0805_2012Metric_Pad1.20x1.40mm_HandSolder" V 5680 5600 50  0001 C CNN
+F 3 "" H 5750 5600 50  0001 C CNN
+	1    5750 5600
+	0    -1   -1   0
+$EndComp

Commit message: Onboard FPGA, passthroughs and a lot of other stuff
Parts:
- added C27: 0.1uF, Capacitor_SMD:C_0805_2012Metric_Pad1.18x1.45mm_HandSolder, symbol bkm-68x-simple-rescue:C_Small
- added C54: 100pF, Capacitor_SMD:C_0805_2012Metric_Pad1.18x1.45mm_HandSolder, symbol bkm-68x-simple-rescue:C_Small
- added C55: 470pF, Capacitor_SMD:C_0805_2012Metric_Pad1.18x1.45mm_HandSolder, symbol bkm-68x-simple-rescue:C_Small
- added J13: PR_R_OUT, BNC-THT:BNC-THT, symbol bkm-68x-simple-rescue:Conn_Coaxial
- added J15: Y_G_OUT, BNC-THT:BNC-THT, symbol bkm-68x-simple-rescue:Conn_Coaxial
- added J16: PB_B_OUT, BNC-THT:BNC-THT, symbol bkm-68x-simple-rescue:Conn_Coaxial
- added J17: EXT_SYNC_OUT, BNC-THT:BNC-THT, symbol bkm-68x-simple-rescue:Conn_Coaxial
- added Q1: MMBT3904, Package_TO_SOT_SMD:SOT-23_Handsoldering, symbol Device:Q_NPN_BEC
- added R80: 100R, Resistor_SMD:R_0805_2012Metric_Pad1.20x1.40mm_HandSolder, symbol bkm-68x-simple-rescue:R
- added R81: 10K, Resistor_SMD:R_0805_2012Metric_Pad1.20x1.40mm_HandSolder, symbol bkm-68x-simple-rescue:R
- added SW3: PR_R_TERM, JS202011SCQN:JS202011SCQN, symbol Switch:SW_DPDT_x2
- added SW4: Y_G_TERM, JS202011SCQN:JS202011SCQN, symbol Switch:SW_DPDT_x2
- added SW5: PB_B_TERM, JS202011SCQN:JS202011SCQN, symbol Switch:SW_DPDT_x2
- added SW6: EXT_SYNC_TERM, JS202011SCQN:JS202011SCQN, symbol Switch:SW_DPDT_x2
- added unit 3 of U1
- added unit 2 of U4
- added unit 3 of U4
- added unit 4 of U4
- C11: value 0.1uF -> 56nF
- R42, R43: value R -> 47R
- R5, R6, R7, R8: value R -> 1K
Connections:
- net labels added: ISL_SD_HD, SYNC_SRC_FILTER
- wire segments 94 -> 99
- no-connect marks 2 -> 1
Other:
- moved on the sheet: C1, C10, C11, C13, C2, C3, C4, C5, C6, C7, C8, C9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

Commit message: Updated some component values
Changed lines of the file:
@@
 P 9600 5050
 F 0 "#PWR031" H 9600 4800 50  0001 C CNN
-F 1 "GNDA" H 9600 4900 50  0000 C CNN
+F 1 "GNDA" H 9750 4950 50  0000 C CNN
 F 2 "" H 9600 5050 50  0001 C CNN
 F 3 "" H 9600 5050 50  0001 C CNN
@@
 U 1 1 6048A8BF
 P 9600 4850
-F 0 "U8" H 9600 5325 50  0000 C CNN
+F 0 "U8" H 9350 4750 50  0000 C CNN
 F 1 "TC7WH125" H 9600 5234 50  0000 C CNN
 F 2 "Package_SO:SSOP-8_2.95x2.8mm_P0.65mm" H 9600 4850 50  0001 C CNN
@@
 U 2 1 604A9430
 P 9600 5650
-F 0 "U8" H 9600 6125 50  0000 C CNN
+F 0 "U8" H 9350 5500 50  0000 C CNN
 F 1 "TC7WH125" H 9600 6034 50  0000 C CNN
 F 2 "Package_SO:SSOP-8_2.95x2.8mm_P0.65mm" H 9600 5650 50  0001 C CNN

Commit message: Replace ADG1611BRUZ with BCPZ
Should also be compatible with Vishay DG1411EEN-T1-GE4
Parts:
- removed U1: ADG1611, Package_SO:TSSOP-16_4.4x5mm_P0.65mm, symbol adg1611:ADG1611
- added U1: ADG1611BCPZ, Package_CSP:LFCSP-16-1EP_4x4mm_P0.65mm_EP2.4x2.4mm, symbol adg1611:ADG1611BCPZ
Other:
- moved on the sheet: C1, C2, J5, J7, R10, R9

Commit message: Rev C1
Parts:
- R11, R13, R9: value 75R -> 150R
- R42, R43: value 47R -> 68R
Changed lines of the file:
@@
 P 8400 2450
 F 0 "R11" V 8480 2450 50  0000 C CNN
-F 1 "75R" V 8400 2450 50  0000 C CNN
+F 1 "150R" V 8400 2450 50  0000 C CNN
 F 2 "Resistor_SMD:R_0805_2012Metric_Pad1.20x1.40mm_HandSolder" V 8330 2450 50  0001 C CNN
 F 3 "" H 8400 2450 50  0001 C CNN
@@
 P 8400 3350
 F 0 "R13" V 8480 3350 50  0000 C CNN
-F 1 "75R" V 8400 3350 50  0000 C CNN
+F 1 "150R" V 8400 3350 50  0000 C CNN
 F 2 "Resistor_SMD:R_0805_2012Metric_Pad1.20x1.40mm_HandSolder" V 8330 3350 50  0001 C CNN
 F 3 "" H 8400 3350 50  0001 C CNN
@@
 P 1900 5500
 F 0 "R43" V 1980 5500 50  0000 C CNN
-F 1 "47R" V 1900 5500 50  0000 C CNN
+F 1 "68R" V 1900 5500 50  0000 C CNN
 F 2 "Resistor_SMD:R_0805_2012Metric_Pad1.20x1.40mm_HandSolder" V 1830 5500 50  0001 C CNN
 F 3 "" H 1900 5500 50  0001 C CNN
@@
 P 4600 5300
 F 0 "R42" V 4680 5300 50  0000 C CNN
-F 1 "47R" V 4600 5300 50  0000 C CNN
+F 1 "68R" V 4600 5300 50  0000 C CNN
 F 2 "Resistor_SMD:R_0805_2012Metric_Pad1.20x1.40mm_HandSolder" V 4530 5300 50  0001 C CNN
 F 3 "" H 4600 5300 50  0001 C CNN
@@
 U 2 1 60A5CDD2
 P 9450 1250
+AR Path="/60A5CDD2" Ref="U1"  Part="2"
+AR Path="/5F1E9444/60A5CDD2" Ref="U1"  Part="2"
 F 0 "U1" H 9450 1747 60  0000 C CNN
 F 1 "ADG1611BCPZ" H 9450 1641 60  0000 C CNN
@@
 U 1 1 60A66CA9
 P 9700 2450
+AR Path="/60A66CA9" Ref="U1"  Part="1"
+AR Path="/5F1E9444/60A66CA9" Ref="U1"  Part="1"
 F 0 "U1" H 9700 2947 60  0000 C CNN
 F 1 "ADG1611BCPZ" H 9700 2841 60  0000 C CNN
@@
 U 4 1 60A7F254
 P 9700 3350
+AR Path="/60A7F254" Ref="U1"  Part="4"
+AR Path="/5F1E9444/60A7F254" Ref="U1"  Part="4"
 F 0 "U1" H 9700 3847 60  0000 C CNN
 F 1 "ADG1611BCPZ" H 9700 3741 60  0000 C CNN
@@
 U 3 1 60A995BC
 P 7050 3500
+AR Path="/60A995BC" Ref="U1"  Part="3"
+AR Path="/5F1E9444/60A995BC" Ref="U1"  Part="3"
 F 0 "U1" H 7050 3997 60  0000 C CNN
 F 1 "ADG1611BCPZ" H 7050 3891 60  0000 C CNN
@@
 P 8150 1250
 F 0 "R9" V 8230 1250 50  0000 C CNN
-F 1 "75R" V 8150 1250 50  0000 C CNN
+F 1 "150R" V 8150 1250 50  0000 C CNN
 F 2 "Resistor_SMD:R_0805_2012Metric_Pad1.20x1.40mm_HandSolder" V 8080 1250 50  0001 C CNN
 F 3 "" H 8150 1250 50  0001 C CNN

Commit message: Revision D
Parts:
- added C62, C63, C64: 0.1uF, Capacitor_SMD:C_0805_2012Metric_Pad1.18x1.45mm_HandSolder, symbol bkm-68x-simple-rescue:C_Small
- added C65: 220pF, Capacitor_SMD:C_0805_2012Metric_Pad1.18x1.45mm_HandSolder, symbol bkm-68x-simple-rescue:C_Small
- added R84: 10K, Resistor_SMD:R_0805_2012Metric_Pad1.20x1.40mm_HandSolder, symbol bkm-68x-simple-rescue:R
- added U16: SN74LVC1G14DBV, Package_TO_SOT_SMD:SOT-23-5, symbol 74xGxx:SN74LVC1G14DBV
- added U17: ISL4089, Package_SO:SOIC-8_3.9x4.9mm_P1.27mm, symbol ISL4089:ISL4089
Connections:
- net +5VA: now also C62.2, C63.1, U16.5 (VCC), U17.8 (V+)
- net GND: now also C62.1, C63.2, R84.2, U16.3 (GND), U17.3 (VREF), U17.5 (GND)
- net Y_G_AMP: now also C64.1; no longer R11.1
- net CSYNC: now reaches U3.1 (CSYNC)
- net CSYNC: now also C65.1
- new net: C65.2, R84.1, U16.2
- new net: C64.2, U17.2 (IN+)
- new net Y_G_NORM: R11.1, U17.1 (IN-), U17.7 (VOUT)
- new net ~CSYNC: U16.4, U17.4 (HOLD)
- no-connect marks 1 -> 0
Other:
- moved on the sheet: J10, J9
Changed lines of the file:
@@
-$EndComp
-$Comp
-L isl59885:ISL59885 U3
-U 1 1 5F267457
-P 3200 5400
-F 0 "U3" H 3200 5850 60  0000 C CNN
-F 1 "ISL59885" H 3200 4950 60  0000 C CNN
-F 2 "Package_SO:SOIC-8_3.9x4.9mm_P1.27mm" H 3200 5400 60  0001 C CNN
-F 3 "" H 3200 5400 60  0001 C CNN
-	1    3200 5400
-	1    0    0    -1
 $EndComp
 $Comp
@@
 ~VIDEO_OE
 Text GLabel 8250 2450 0    60   Input ~ 0
-Y_G_AMP
+Y_G_NORM
 Text GLabel 8250 3350 0    60   Input ~ 0
 PB_B_AMP
@@
 	1    0    0    1
 $EndComp
-NoConn ~ 2650 5100
 $Comp
 L bkm-68x-simple-rescue:R R10
@@
 L bkm-68x-simple-rescue:TEST_1P J9
 U 1 1 5F2887BD
-P 6050 6950
-F 0 "J9" H 6050 7220 50  0000 C CNN
-F 1 "TP_INT_EXT_SYNC" H 6050 7150 50  0000 C CNN
-F 2 "TestPoint:TestPoint_Pad_D2.0mm" H 6250 6950 50  0001 C CNN
-F 3 "" H 6250 6950 50  0001 C CNN
-	1    6050 6950
-	1    0    0    -1
-$EndComp
-Text GLabel 6650 6950 3    60   Input ~ 0
+P 7850 6100
+F 0 "J9" V 7950 6250 50  0000 C CNN
+F 1 "TP_INT_EXT_SYNC" V 7850 6600 50  0000 C CNN
+F 2 "TestPoint:TestPoint_Pad_D2.0mm" H 8050 6100 50  0001 C CNN
+F 3 "" H 8050 6100 50  0001 C CNN
+	1    7850 6100
+	0    -1   -1   0
+$EndComp
+Text GLabel 7850 6350 2    60   Input ~ 0
 ~VIDEO_OE
 $Comp
 L bkm-68x-simple-rescue:TEST_1P J10
 U 1 1 5F288DE7
-P 6650 6950
-F 0 "J10" H 6650 7220 50  0000 C CNN
-F 1 "TP_VIDEO_OE" H 6650 7150 50  0000 C CNN
-F 2 "TestPoint:TestPoint_Pad_D2.0mm" H 6850 6950 50  0001 C CNN
-F 3 "" H 6850 6950 50  0001 C CNN
-	1    6650 6950
-	1    0    0    -1
+P 7850 6350
+F 0 "J10" V 7950 6500 50  0000 C CNN
+F 1 "TP_VIDEO_OE" V 7850 6800 50  0000 C CNN
+F 2 "TestPoint:TestPoint_Pad_D2.0mm" H 8050 6350 50  0001 C CNN
+F 3 "" H 8050 6350 50  0001 C CNN
+	1    7850 6350
+	0    -1   -1   0
 $EndComp
 Wire Wire Line
@@
 Text GLabel 10800 4750 3    60   Input ~ 0
 HSYNC
-Text GLabel 6050 6950 3    60   Input ~ 0
+Text GLabel 7850 6100 2    60   Input ~ 0
 INT_~EXT~_SYNC
 $Comp
@@
 Wire Wire Line
 	8600 2450 9250 2450
+$Comp
+L 74xGxx:SN74LVC1G14DBV U16
+U 1 1 60ED24FD
+P 5150 4300
+F 0 "U16" H 5300 4500 50  0000 L CNN
+F 1 "SN74LVC1G14DBV" H 5350 4150 50  0000 L CNN
+F 2 "Package_TO_SOT_SMD:SOT-23-5" H 5150 4050 50  0001 C CNN
+F 3 "http://www.ti.com/lit/ds/symlink/sn74lvc1g14.pdf" H 5150 4300 50  0001 C CNN
+	1    5150 4300
+	1    0    0    -1
+$EndComp
+$Comp
+L power:GNDA #PWR0271
+U 1 1 60ED4879
+P 5150 4500
+F 0 "#PWR0271" H 5150 4250 50  0001 C CNN
+F 1 "GNDA" H 5150 4350 50  0000 C CNN
+F 2 "" H 5150 4500 50  0001 C CNN
+F 3 "" H 5150 4500 50  0001 C CNN
+	1    5150 4500
+	1    0    0    -1
+$EndComp
+$Comp
+L power:+5VA #PWR0272
+U 1 1 60ED6EE9
+P 5150 3950
+F 0 "#PWR0272" H 5150 3800 50  0001 C CNN
+F 1 "+5VA" V 5150 4150 50  0000 C CNN
+F 2 "" H 5150 3950 50  0001 C CNN
+F 3 "" H 5150 3950 50  0001 C CNN
+	1    5150 3950
+	-1   0    0    -1
+$EndComp
+Wire Wire Line
+	5150 3950 5150 4050
+$Comp
+L isl59885:ISL59885 U3
+U 1 1 5F267457
+P 3200 5400
+F 0 "U3" H 3200 5850 60  0000 C CNN
+F 1 "ISL59885" H 3200 4950 60  0000 C CNN
+F 2 "Package_SO:SOIC-8_3.9x4.9mm_P1.27mm" H 3200 5400 60  0001 C CNN
+F 3 "" H 3200 5400 60  0001 C CNN
+	1    3200 5400
+	1    0    0    -1
+$EndComp
+Text Label 2650 5100 2    50   ~ 0
+CSYNC
+Text Label 4600 4300 2    50   ~ 0
+CSYNC
+$Comp
+L bkm-68x-simple-rescue:C_Small C62
+U 1 1 60EE65D1
+P 4900 4050
+F 0 "C62" V 4950 3900 50  0000 L CNN
+F 1 "0.1uF" V 4800 3900 50  0000 L CNN
+F 2 "Capacitor_SMD:C_0805_2012Metric_Pad1.18x1.45mm_HandSolder" H 4900 4050 50  0001 C CNN
+F 3 "" H 4900 4050 50  0001 C CNN
+	1    4900 4050
+	0    -1   -1   0
+$EndComp
+Wire Wire Line
+	5000 4050 5150 4050
+Connection ~ 5150 4050
+Wire Wire Line
+	5150 4050 5150 4100
+$Comp
+L power:GNDA #PWR0273
+U 1 1 60EEA591
+P 4800 4050
+F 0 "#PWR0273" H 4800 3800 50  0001 C CNN
+F 1 "GNDA" V 4800 3850 50  0000 C CNN
+F 2 "" H 4800 4050 50  0001 C CNN
+F 3 "" H 4800 4050 50  0001 C CNN
+	1    4800 4050
+	0    1    1    0
+$EndComp
+Text Label 5450 4300 0    50   ~ 0
+~CSYNC
+$Comp
+L ISL4089:ISL4089 U17
+U 1 1 60F6B901
+P 5600 6800
+F 0 "U17" H 5600 7347 60  0000 C CNN
+F 1 "ISL4089" H 5600 7241 60  0000 C CNN
+F 2 "Package_SO:SOIC-8_3.9x4.9mm_P1.27mm" H 5600 6800 60  0001 C CNN
+F 3 "" H 5600 6800 60  0001 C CNN
+	1    5600 6800
+	1    0    0    -1
+$EndComp
+$Comp
+L power:GNDA #PWR0274
+U 1 1 60F6DCD2
+P 5100 6900
+F 0 "#PWR0274" H 5100 6650 50  0001 C CNN
+F 1 "GNDA" V 5100 6700 50  0000 C CNN
+F 2 "" H 5100 6900 50  0001 C CNN
+F 3 "" H 5100 6900 50  0001 C CNN
+	1    5100 6900
+	0    1    1    0
+$EndComp
+$Comp
+L power:GNDA #PWR0275
+U 1 1 60F6FA2B
+P 6100 7100
+F 0 "#PWR0275" H 6100 6850 50  0001 C CNN
+F 1 "GNDA" V 6100 6900 50  0000 C CNN
+F 2 "" H 6100 7100 50  0001 C CNN
+F 3 "" H 6100 7100 50  0001 C CNN
+	1    6100 7100
+	0    -1   -1   0
+$EndComp
+Wire Wire Line
+	5100 6500 5050 6500
+Wire Wire Line
+	5050 6500 5050 6200
+Wire Wire Line
+	5050 6200 6200 6200
+Wire Wire Line
+	6200 6200 6200 6700
+Wire Wire Line
+	6200 6700 6100 6700
+$Comp
+L bkm-68x-simple-rescue:R R84
+U 1 1 60F7BE6C
+P 4850 4500
+F 0 "R84" V 4930 4500 50  0000 C CNN
+F 1 "10K" V 4850 4500 50  0000 C CNN
+F 2 "Resistor_SMD:R_0805_2012Metric_Pad1.20x1.40mm_HandSolder" V 4780 4500 50  0001 C CNN
+F 3 "" H 4850 4500 50  0001 C CNN
+	1    4850 4500
+	1    0    0    -1
+$EndComp
+$Comp
+L bkm-68x-simple-rescue:C_Small C65
+U 1 1 60F7D5A8
+P 4700 4300
+F 0 "C65" V 4750 4150 50  0000 L CNN
+F 1 "220pF" V 4600 4150 50  0000 L CNN
+F 2 "Capacitor_SMD:C_0805_2012Metric_Pad1.18x1.45mm_HandSolder" H 4700 4300 50  0001 C CNN
+F 3 "" H 4700 4300 50  0001 C CNN
+	1    4700 4300
+	0    -1   -1   0
+$EndComp
+Wire Wire Line
+	4800 4300 4850 4300
+Wire Wire Line
+	4850 4350 4850 4300
+Connection ~ 4850 4300
+$Comp
+L power:GNDA #PWR0276
+U 1 1 60FABEE7
+P 4850 4650
+F 0 "#PWR0276" H 4850 4400 50  0001 C CNN
+F 1 "GNDA" H 4850 4500 50  0000 C CNN
+F 2 "" H 4850 4650 50  0001 C CNN
+F 3 "" H 4850 4650 50  0001 C CNN
+	1    4850 4650
+	1    0    0    -1
+$EndComp
+Text GLabel 4900 6700 0    60   Input ~ 0
+Y_G_AMP
+$Comp
+L bkm-68x-simple-rescue:C_Small C64
+U 1 1 60FB4442
+P 5000 6700
+F 0 "C64" V 5050 6550 50  0000 L CNN
+F 1 "0.1uF" V 4900 6550 50  0000 L CNN
+F 2 "Capacitor_SMD:C_0805_2012Metric_Pad1.18x1.45mm_HandSolder" H 5000 6700 50  0001 C CNN
+F 3 "" H 5000 6700 50  0001 C CNN
+	1    5000 6700
+	0    -1   -1   0
+$EndComp
+$Comp
+L power:+5VA #PWR0277
+U 1 1 60FC0697
+P 6350 6500
+F 0 "#PWR0277" H 6350 6350 50  0001 C CNN
+F 1 "+5VA" V 6350 6700 50  0000 C CNN
+F 2 "" H 6350 6500 50  0001 C CNN
+F 3 "" H 6350 6500 50  0001 C CNN
+	1    6350 6500
+	0    1    -1   0
+$EndComp
+Wire Wire Line
+	6100 6500 6300 6500
+$Comp
+L bkm-68x-simple-rescue:C_Small C63
+U 1 1 60FC685F
+P 6300 6300
+F 0 "C63" V 6350 6150 50  0000 L CNN
+F 1 "0.1uF" V 6200 6150 50  0000 L CNN
+F 2 "Capacitor_SMD:C_0805_2012Metric_Pad1.18x1.45mm_HandSolder" H 6300 6300 50  0001 C CNN
+F 3 "" H 6300 6300 50  0001 C CNN
+	1    6300 6300
+	-1   0    0    1
+$EndComp
+$Comp
+L power:GNDA #PWR0278
+U 1 1 60FC7BA2
+P 6300 6200
+F 0 "#PWR0278" H 6300 5950 50  0001 C CNN
+F 1 "GNDA" V 6300 6000 50  0000 C CNN
+F 2 "" H 6300 6200 50  0001 C CNN
+F 3 "" H 6300 6200 50  0001 C CNN
+	1    6300 6200
+	-1   0    0    1
+$EndComp
+Wire Wire Line
+	6300 6400 6300 6500
+Wire Wire Line
+	6300 6500 6350 6500
+Text GLabel 6250 6700 2    60   Input ~ 0
+Y_G_NORM
+Wire Wire Line
+	6200 6700 6250 6700
+Connection ~ 6200 6700
+Connection ~ 6300 6500
+Wire Wire Line
+	4850 4300 4950 4300
+Text Label 5100 7100 2    50   ~ 0
+~CSYNC
 $EndSCHEMATC

Commit message: Rev. E
Parts:
- removed R42, R43: 68R, Resistor_SMD:R_0805_2012Metric_Pad1.20x1.40mm_HandSolder, symbol bkm-68x-simple-rescue:R
- added C69: NM, Capacitor_SMD:C_0805_2012Metric_Pad1.18x1.45mm_HandSolder, symbol bkm-68x-simple-rescue:C_Small
- added R89: NM, Resistor_SMD:R_0805_2012Metric_Pad1.20x1.40mm_HandSolder, symbol bkm-68x-simple-rescue:R
- added R90: 0R, Resistor_SMD:R_0805_2012Metric_Pad1.20x1.40mm_HandSolder, symbol bkm-68x-simple-rescue:R
Connections:
- net +5VA: now also R89.1
- net -5VA: no longer C8.1, U4.5 (VSS), U4.5 (VSS), U4.5 (VSS), U4.5 (VSS)
- net EXT_SYNC_AMP: now also U4.9 (SA); no longer U4.2 (SA)
- net GND: now also C69.1, R90.2; no longer R7.2, R8.2, U17.3 (VREF), U4.10 (IN), U4.7 (SB), U4.9 (SA)
- net HSYNC_SEP: now also U3.7 (HSYNC)
- net INT_~EXT~_SYNC: now also U4.10 (IN); no longer U4.1 (IN)
- net SYNC_SRC: now also U4.8 (D); no longer U4.3 (D)
- net VSYNC_SEP: now also U3.3 (VSYNC)
- net Y_G_AMP: now also U4.2 (SA), U4.7 (SB); no longer U4.4 (SB)
- net Y_G_NORM: now also U4.4 (SB); no longer R11.1
- net at R6.2: no longer U3.3 (VSYNC)
- net at R5.1: no longer U3.7 (HSYNC)
- net at R6.1: no longer R8.1
- net at R5.2: no longer R7.1
- new net: C69.2, R89.2, R90.1, U17.3 (VREF)
- new net -1.5V: C8.1, U4.5 (VSS), U4.5 (VSS), U4.5 (VSS), U4.5 (VSS)
- new net NORM_Y_G: U4.1 (IN)
- new net Y_G_SW: R11.1, U4.3 (D)
Other:
- moved on the sheet: C10, C11, C27, C62, C63, C64, C65, C8, D1, D2, D3, D4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
