File: bkm-68x-video.sch (KiCad schematic (older format))
At the start: 76 parts, among them J1 PR_R, J10 TP_VIDEO_OE, J11 TP_VSYNC, J13 PR_R_OUT, J15 Y_G_OUT, J16 PB_B_OUT, J17 EXT_SYNC_OUT, J2 Y_G, J3 PB_B, J4 EXT_SYNC, J5 TP_Y_G, J6 TP_PB_B, J7 TP_PR_R, J8 TP_HSYNC, J9 TP_INT_EXT_SYNC, Q1 MMBT3904, SW3 PR_R_TERM, SW4 Y_G_TERM, SW5 PB_B_TERM, SW6 EXT_SYNC_TERM, U1 ADG1611BCPZ, U16 SN74LVC1G14DBV, U17 ISL4089, U2 THS7374, U3 ISL59885, U4 ADG734, U8 TC7WH125

Commit message: Rev. E1
Parts:
- removed C8: 0.1uF, Capacitor_SMD:C_0805_2012Metric_Pad1.18x1.45mm_HandSolder, symbol bkm-68x-simple-rescue:C_Small
- removed R5, R6, R7, R8: 1K, Resistor_SMD:R_0805_2012Metric_Pad1.20x1.40mm_HandSolder, symbol bkm-68x-simple-rescue:R
- D1, D2, D3, D4, D5, D6, D7, D8: value D_ESD -> NM
Connections:
- net -1.5V is gone; now on net GND: U4.5 (VSS), U4.5 (VSS), U4.5 (VSS), U4.5 (VSS)
Changed lines of the file:
@@
 Text GLabel 2000 5450 0    60   Input ~ 0
 VSYNC_SEP
-$Comp
-L bkm-68x-simple-rescue:R R5
-U 1 1 5F26786D
-P 800 6100
-F 0 "R5" V 880 6100 50  0000 C CNN
-F 1 "1K" V 800 6100 50  0000 C CNN
-F 2 "Resistor_SMD:R_0805_2012Metric_Pad1.20x1.40mm_HandSolder" V 730 6100 50  0001 C CNN
-F 3 "" H 800 6100 50  0001 C CNN
-	1    800  6100
-	0    -1   -1   0
-$EndComp
-$Comp
-L bkm-68x-simple-rescue:R R7
-U 1 1 5F2678B9
-P 700 5750
-F 0 "R7" V 780 5750 50  0000 C CNN
-F 1 "1K" V 700 5750 50  0000 C CNN
-F 2 "Resistor_SMD:R_0805_2012Metric_Pad1.20x1.40mm_HandSolder" V 630 5750 50  0001 C CNN
-F 3 "" H 700 5750 50  0001 C CNN
-	1    700  5750
-	1    0    0    -1
-$EndComp
 Wire Wire Line
 	3250 5250 3450 5250
@@
 P 1200 1800
 F 0 "D1" H 1150 1880 50  0000 L CNN
-F 1 "D_ESD" H 1050 1720 50  0000 L CNN
+F 1 "NM" H 1050 1720 50  0000 L CNN
 F 2 "Diode_SMD:D_SOD-123" V 1200 1800 50  0001 C CNN
 F 3 "" V 1200 1800 50  0001 C CNN
@@
 P 1200 2100
 F 0 "D2" H 1150 2180 50  0000 L CNN
-F 1 "D_ESD" H 1050 2020 50  0000 L CNN
+F 1 "NM" H 1050 2020 50  0000 L CNN
 F 2 "Diode_SMD:D_SOD-123" V 1200 2100 50  0001 C CNN
 F 3 "" V 1200 2100 50  0001 C CNN
@@
 P 1200 800
 F 0 "D5" H 1150 880 50  0000 L CNN
-F 1 "D_ESD" H 1050 720 50  0000 L CNN
+F 1 "NM" H 1050 720 50  0000 L CNN
 F 2 "Diode_SMD:D_SOD-123" V 1200 800 50  0001 C CNN
 F 3 "" V 1200 800 50  0001 C CNN
@@
 P 1200 1100
 F 0 "D6" H 1150 1180 50  0000 L CNN
-F 1 "D_ESD" H 1050 1020 50  0000 L CNN
+F 1 "NM" H 1050 1020 50  0000 L CNN
 F 2 "Diode_SMD:D_SOD-123" V 1200 1100 50  0001 C CNN
 F 3 "" V 1200 1100 50  0001 C CNN
@@
 P 1200 4150
 F 0 "D8" H 1150 4230 50  0000 L CNN
-F 1 "D_ESD" H 1050 4070 50  0000 L CNN
+F 1 "NM" H 1050 4070 50  0000 L CNN
 F 2 "Diode_SMD:D_SOD-123" V 1200 4150 50  0001 C CNN
 F 3 "" V 1200 4150 50  0001 C CNN
@@
 Connection ~ 6750 1600
 $Comp
-L bkm-68x-simple-rescue:C_Small C8
-U 1 1 5F27113B
-P 7150 4550
-F 0 "C8" V 7200 4400 50  0000 L CNN
-F 1 "0.1uF" V 7050 4400 50  0000 L CNN
-F 2 "Capacitor_SMD:C_0805_2012Metric_Pad1.18x1.45mm_HandSolder" H 7150 4550 50  0001 C CNN
-F 3 "" H 7150 4550 50  0001 C CNN
-	1    7150 4550
-	0    1    1    0
-$EndComp
-$Comp
 L bkm-68x-simple-rescue:C_Small C9
 U 1 1 5F2711E5
@@
 	1    7750 4500
 	0    -1   -1   0
-$EndComp
-$Comp
-L power:GNDA #PWR025
-U 1 1 5F271595
-P 7050 4550
-F 0 "#PWR025" H 7050 4300 50  0001 C CNN
-F 1 "GNDA" V 7050 4350 50  0000 C CNN
-F 2 "" H 7050 4550 50  0001 C CNN
-F 3 "" H 7050 4550 50  0001 C CNN
-	1    7050 4550
-	0    1    1    0
 $EndComp
 $Comp
@@
 P 1200 3850
 F 0 "D7" H 1150 3930 50  0000 L CNN
-F 1 "D_ESD" H 1050 3770 50  0000 L CNN
+F 1 "NM" H 1050 3770 50  0000 L CNN
 F 2 "Diode_SMD:D_SOD-123" V 1200 3850 50  0001 C CNN
 F 3 "" V 1200 3850 50  0001 C CNN
@@
 P 1200 3100
 F 0 "D4" H 1150 3180 50  0000 L CNN
-F 1 "D_ESD" H 1050 3020 50  0000 L CNN
+F 1 "NM" H 1050 3020 50  0000 L CNN
 F 2 "Diode_SMD:D_SOD-123" V 1200 3100 50  0001 C CNN
 F 3 "" V 1200 3100 50  0001 C CNN
@@
 P 1200 2800
 F 0 "D3" H 1150 2880 50  0000 L CNN
-F 1 "D_ESD" H 1050 2720 50  0000 L CNN
+F 1 "NM" H 1050 2720 50  0000 L CNN
 F 2 "Diode_SMD:D_SOD-123" V 1200 2800 50  0001 C CNN
 F 3 "" V 1200 2800 50  0001 C CNN
@@
 Text GLabel 4950 5600 0    60   Input ~ 0
 NORM_Y_G
-Text GLabel 7250 4550 1    50   Input ~ 0
--1.5V
-Text GLabel 5350 4550 1    50   Input ~ 0
--1.5V
-Text GLabel 2450 6400 1    50   Input ~ 0
--1.5V
-Text GLabel 1350 6400 1    50   Input ~ 0
--1.5V
 $Comp
 L bkm-68x-simple-rescue:R R89
@@
 	3800 7000 4550 7000
 $Comp
-L bkm-68x-simple-rescue:R R6
-U 1 1 5F2676DF
-P 850 5500
-F 0 "R6" V 930 5500 50  0000 C CNN
-F 1 "1K" V 850 5500 50  0000 C CNN
-F 2 "Resistor_SMD:R_0805_2012Metric_Pad1.20x1.40mm_HandSolder" V 780 5500 50  0001 C CNN
-F 3 "" H 850 5500 50  0001 C CNN
-	1    850  5500
-	0    -1   -1   0
-$EndComp
-$Comp
-L bkm-68x-simple-rescue:R R8
-U 1 1 5F267738
-P 1000 5750
-F 0 "R8" V 1080 5750 50  0000 C CNN
-F 1 "1K" V 1000 5750 50  0000 C CNN
-F 2 "Resistor_SMD:R_0805_2012Metric_Pad1.20x1.40mm_HandSolder" V 930 5750 50  0001 C CNN
-F 3 "" H 1000 5750 50  0001 C CNN
-	1    1000 5750
-	1    0    0    -1
+L power:GNDA #PWR0153
+U 1 1 61223D8E
+P 2450 6400
+F 0 "#PWR0153" H 2450 6150 50  0001 C CNN
+F 1 "GNDA" V 2450 6200 50  0000 C CNN
+F 2 "" H 2450 6400 50  0001 C CNN
+F 3 "" H 2450 6400 50  0001 C CNN
+	1    2450 6400
+	-1   0    0    1
+$EndComp
+$Comp
+L power:GNDA #PWR0282
+U 1 1 612243E8
+P 1350 6400
+F 0 "#PWR0282" H 1350 6150 50  0001 C CNN
+F 1 "GNDA" V 1350 6200 50  0000 C CNN
+F 2 "" H 1350 6400 50  0001 C CNN
+F 3 "" H 1350 6400 50  0001 C CNN
+	1    1350 6400
+	-1   0    0    1
+$EndComp
+$Comp
+L power:GNDA #PWR0283
+U 1 1 61227169
+P 5350 4550
+F 0 "#PWR0283" H 5350 4300 50  0001 C CNN
+F 1 "GNDA" V 5350 4350 50  0000 C CNN
+F 2 "" H 5350 4550 50  0001 C CNN
+F 3 "" H 5350 4550 50  0001 C CNN
+	1    5350 4550
+	-1   0    0    1
+$EndComp
+$Comp
+L power:GNDA #PWR0284
+U 1 1 612279B8
+P 7250 4550
+F 0 "#PWR0284" H 7250 4300 50  0001 C CNN
+F 1 "GNDA" V 7250 4350 50  0000 C CNN
+F 2 "" H 7250 4550 50  0001 C CNN
+F 3 "" H 7250 4550 50  0001 C CNN
+	1    7250 4550
+	-1   0    0    1
 $EndComp
 $EndSCHEMATC
