File: bkm-68x-simple.kicad_pcb (KiCad board)
At the start: 2 copper layers, 230.4 x 233.5 mm, 201 parts, among them CN985 mezz-conn-02x50, CN986 mezz-conn-02x50, J1 PR_R, J10 TP_VIDEO_OE, J11 TP_VSYNC, J12 JTAG, J13 PR_R_OUT, J14 JTAG, J15 Y_G_OUT, J16 PB_B_OUT, J17 EXT_SYNC_OUT, J2 Y_G, J3 PB_B, J4 EXT_SYNC, J5 TP_Y_G, J6 TP_PB_B, J7 TP_PR_R, J8 TP_HSYNC, J9 TP_INT_EXT_SYNC, Q1 MMBT3904, SW1 FORCE_VIDEO, SW2 FORCE_VIDEO, SW3 PR_R_TERM, SW4 Y_G_TERM, SW5 PB_B_TERM, SW6 EXT_SYNC_TERM, U1 ADG1611BCPZ, U10 74LVC541A, U11 BA33BC0FP-E2, U12 TC7SZ125FU, U13 LM2990SX-5.0, U14 BA50BC0FP-E2, U15 10M08SC, U2 THS7374, U3 ISL59885, U4 ADG734, U5 74LVC14A, U6 74LVC14A, U7 74LVC14A, U8 TC7WH125, U9 KC2520Z50

Commit message: Revision D
Parts:
- added C62: 0.1uF, Capacitor_SMD:C_0805_2012Metric_Pad1.18x1.45mm_HandSolder, F.Cu at (214.6, 91.8)
- added C63: 0.1uF, Capacitor_SMD:C_0805_2012Metric_Pad1.18x1.45mm_HandSolder, F.Cu at (221.0, 81.5)
- added C64: 0.1uF, Capacitor_SMD:C_0805_2012Metric_Pad1.18x1.45mm_HandSolder, F.Cu at (215.2, 86.2)
- added C65: 220pF, Capacitor_SMD:C_0805_2012Metric_Pad1.18x1.45mm_HandSolder, F.Cu at (217.2, 96.6)
- added R84: 10K, Resistor_SMD:R_0805_2012Metric_Pad1.20x1.40mm_HandSolder, F.Cu at (218.2, 93.6)
- added U16: SN74LVC1G14DBV, Package_TO_SOT_SMD:SOT-23-5, F.Cu at (217.5, 90.6)
- added U17: ISL4089, Package_SO:SOIC-8_3.9x4.9mm_P1.27mm, F.Cu at (220.9, 85.5)
- H1, H2: value SCREWMOUNT_90DEG -> Keystone 7794
Connections:
- R11 pad 1: Y_G_AMP -> Y_G_NORM
- U3 pad 1: (no net) -> /Video/CSYNC
Routing:
- net /Video/CSYNC: track 0.00 -> 30.4 mm, vias 0 -> 4
- net Y_G_AMP: track 63.5 -> 35.6 mm
- net Y_G_NORM: track 0.00 -> 24.6 mm
- net Net-(C65-Pad2): track 0.00 -> 4.03 mm
- net +5VA: track 533.8 -> 537.7 mm, vias 11 -> 13
- net Net-(C64-Pad2): track 0.00 -> 3.42 mm
- net /Video/~CSYNC: track 0.00 -> 2.10 mm
- net GND: track 164.7 -> 166.1 mm, vias 57 -> 58
- net PB_B_AMP: track 52.3 -> 53.6 mm
- net /Video/ISL_SD_HD: track 10.8 -> 11.5 mm
Other:
- board text added: "Rev. D"
- board text removed: "Rev. C1"

Commit message: Revision D1
Parts:
- added J18: Conn_01x02_Male, Connector_PinHeader_2.54mm:PinHeader_1x02_P2.54mm_Vertical, F.Cu at (264.4, 194.2)
Other:
- board text added: "GND"
- board text added: "Rev. D1"
- board text added: "STBY_5V"
- board text removed: "Rev. D"

Commit message: Rev. E
Parts:
- removed R5, R6, R7, R8: 1K, Resistor_SMD:R_0805_2012Metric_Pad1.20x1.40mm_HandSolder
- added C66: 2.2uF, Capacitor_SMD:C_0805_2012Metric_Pad1.18x1.45mm_HandSolder, F.Cu at (168.9, 109.0)
- added C67: 2.2uF, Capacitor_SMD:C_0805_2012Metric_Pad1.18x1.45mm_HandSolder, F.Cu at (172.2, 106.0)
- added C68: 10uF, Capacitor_SMD:C_0805_2012Metric_Pad1.18x1.45mm_HandSolder, F.Cu at (157.7, 108.3)
- added C69: NM, Capacitor_SMD:C_0805_2012Metric_Pad1.18x1.45mm_HandSolder, F.Cu at (199.3, 103.1)
- added C70: 10uF, Capacitor_SMD:C_0805_2012Metric_Pad1.18x1.45mm_HandSolder, F.Cu at (201.5, 93.4)
- added C71: 0.1uF, Capacitor_SMD:C_0805_2012Metric_Pad1.18x1.45mm_HandSolder, F.Cu at (197.5, 183.4)
- added J19: TP_NORM_Y_G, TestPoint:TestPoint_Pad_D2.0mm, F.Cu at (183.2, 126.3)
- added J20: TP_RGB_COMP_X, TestPoint:TestPoint_Pad_D2.0mm, F.Cu at (177.8, 241.6)
- added J21: TP_HD_SD_X, TestPoint:TestPoint_Pad_D2.0mm, F.Cu at (174.5, 237.0)
- added R85: 22,1K 0,1%, Resistor_SMD:R_0805_2012Metric_Pad1.20x1.40mm_HandSolder, F.Cu at (175.5, 109.0)
- added R86: 82,5K 0.1%, Resistor_SMD:R_0805_2012Metric_Pad1.20x1.40mm_HandSolder, F.Cu at (174.5, 112.0)
- added R87: 22R, Resistor_SMD:R_0805_2012Metric_Pad1.20x1.40mm_HandSolder, F.Cu at (191.8, 184.6)
- added R88: 22R, Resistor_SMD:R_0805_2012Metric_Pad1.20x1.40mm_HandSolder, F.Cu at (175.4, 205.8)
- added R89: NM, Resistor_SMD:R_0805_2012Metric_Pad1.20x1.40mm_HandSolder, F.Cu at (191.0, 98.9)
- added R90: 0R, Resistor_SMD:R_0805_2012Metric_Pad1.20x1.40mm_HandSolder, F.Cu at (199.3, 101.1)
- added U18: TPS72301, Package_TO_SOT_SMD:SOT-23-5, F.Cu at (172.2, 109.0)
- added U19: 74LVC2G34, Package_TO_SOT_SMD:SOT-23-6_Handsoldering, F.Cu at (201.2, 179.7)
- moved C7 41.2 mm to (157.7, 105.5), turned to 0 degrees
- moved C3 34.9 mm to (148.5, 97.4)
- moved C4 34.9 mm to (148.5, 99.6)
- moved C5 34.9 mm to (148.4, 101.7)
- moved C6 34.9 mm to (148.4, 103.9)
- moved U2 34.9 mm to (157.7, 101.6)
- moved C62 26.3 mm to (191.1, 103.7)
- moved R84 26.3 mm to (194.7, 105.5)
- moved U16 26.3 mm to (194.0, 102.4)
- moved U17 26.3 mm to (197.4, 97.3)
- moved C63 26.3 mm to (197.5, 93.4)
- moved C64 26.3 mm to (191.0, 96.7), turned to 0 degrees
- moved C65 25.0 mm to (194.7, 107.6), turned to 180 degrees
- moved C8 17.9 mm to (173.4, 102.3)
- moved C9 17.0 mm to (185.8, 102.3), turned to 180 degrees
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Connections:
- C8 pad 1: -5VA -> -1.5V
- R11 pad 1: Y_G_NORM -> Y_G_SW
- R42 pad 1: Net-(R42-Pad1) -> HSYNC_SEP_BUF
- R42 pad 2: HSYNC_SEP -> Net-(R42-Pad2)
- R43 pad 1: VSYNC_SEP -> VSYNC_SEP_BUF
- U15 pad 30: INT_~EXT~_SYNC -> Net-(R87-Pad1)
- U15 pad 33: (no net) -> Net-(R88-Pad1)
- U15 pad 44: (no net) -> RGB_COMP_X
- U15 pad 50: (no net) -> HD_SD_X
- U15 pad 6: HSYNC_SEP -> HSYNC_SEP_BUF
- U15 pad 8: VSYNC_SEP -> VSYNC_SEP_BUF
- U17 pad 3: GND -> Net-(C69-Pad2)
- U3 pad 3: Net-(R6-Pad2) -> VSYNC_SEP
- U3 pad 7: Net-(R5-Pad1) -> HSYNC_SEP
- U4 pad 1: INT_~EXT~_SYNC -> NORM_Y_G
- U4 pad 10: GND -> INT_~EXT~_SYNC
- U4 pad 2: EXT_SYNC_AMP -> Y_G_AMP
- U4 pad 3: SYNC_SRC -> Y_G_SW
- U4 pad 4: Y_G_AMP -> Y_G_NORM
- U4 pad 5: -5VA -> -1.5V
- U4 pad 7: GND -> Y_G_AMP
- U4 pad 8: (no net) -> SYNC_SRC
- U4 pad 9: GND -> EXT_SYNC_AMP
Routing:
- net NORM_Y_G: track 0.00 -> 137.6 mm, vias 0 -> 2
- net -6V: track 116.5 -> 212.0 mm, vias 1 -> 2
- net +5VA: track 537.7 -> 624.2 mm
- net HSYNC_SEP: track 14.1 -> 97.9 mm
- net Y_G_SW: track 0.00 -> 82.5 mm
- net -5VA: track 116.3 -> 47.8 mm, vias 3 -> 2
- net Net-(R42-Pad1): track 67.2 -> 0.00 mm
- net Net-(R43-Pad2): track 67.2 -> 8.27 mm
- net VSYNC_SEP: track 14.0 -> 71.0 mm
- net PR_R_AMP: track 54.5 -> 89.7 mm
- net PB_B_AMP: track 53.6 -> 87.5 mm, vias 0 -> 2
- net RGB_COMP_X: track 0.00 -> 33.0 mm, vias 0 -> 2
- net HD_SD_X: track 0.00 -> 27.3 mm, vias 0 -> 2
- net INT_~EXT~_SYNC: track 113.2 -> 85.9 mm, vias 4 -> 0
- net Net-(R87-Pad1): track 0.00 -> 25.7 mm, vias 0 -> 2
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Other:
- board text added: "HD_SD_X"
- board text added: "NORM_Y_G"
- board text added: "RGB_COMP_X"
- board text added: "Rev. E1"
- board text added: "~INT~_EXT_SYNC"
- board text removed: "INT_~EXT~_SYNC"
- board text removed: "Rev. D1"

Commit message: Rev. E1
Parts:
- removed C66, C67: 2.2uF, Capacitor_SMD:C_0805_2012Metric_Pad1.18x1.45mm_HandSolder
- removed C8: 0.1uF, Capacitor_SMD:C_0805_2012Metric_Pad1.18x1.45mm_HandSolder
- removed R85: 22,1K 0,1%, Resistor_SMD:R_0805_2012Metric_Pad1.20x1.40mm_HandSolder
- removed R86: 82,5K 0.1%, Resistor_SMD:R_0805_2012Metric_Pad1.20x1.40mm_HandSolder
- removed U18: TPS72301, Package_TO_SOT_SMD:SOT-23-5
- D1, D2, D3, D4, D5, D6, D7, D8: value D_ESD -> NM
- D10, D11, D12, D9: value D_Schottky -> NM
Connections:
- U4 pad 5: -1.5V -> GND
Routing:
- net -6V: track 212.0 -> 116.5 mm, vias 2 -> 1
- net +5VA: track 624.2 -> 593.0 mm, vias 13 -> 14
- net -1.5V: track 11.2 -> 0.00 mm, vias 2 -> 0
- net Net-(R85-Pad2): track 4.23 -> 0.00 mm
- net NORM_Y_G: track 137.6 -> 134.2 mm
- net GND: track 164.3 -> 163.0 mm, vias 62 -> 63
- net Y_G_AMP: track 44.3 -> 43.6 mm

Commit message: Rev. F1
Parts:
- removed C30, C34: 0.1uF, Capacitor_SMD:C_0603_1608Metric_Pad1.08x0.95mm_HandSolder
- removed C50, C51, C52, C53: 10pF, Capacitor_SMD:C_0603_1608Metric_Pad1.08x0.95mm_HandSolder
- removed D11, D12: NM, Diode_SMD:D_SOD-123
- removed R44, R45, R73, R74, R75: 10K, Resistor_SMD:R_0805_2012Metric_Pad1.20x1.40mm_HandSolder
- removed R76: 1K, Resistor_SMD:R_0805_2012Metric_Pad1.20x1.40mm_HandSolder
- removed U15: 10M08SC, Package_QFP:EQFP-144-1EP_20x20mm_P0.5mm_EP8.93x8.7mm_ThermalVias
- removed U4: ADG734, Package_SO:TSSOP-20_4.4x6.5mm_P0.65mm
- added C111: 1uF, Capacitor_SMD:C_0805_2012Metric_Pad1.18x1.45mm_HandSolder, F.Cu at (236.8, 181.2)
- added C112: 1uF, Capacitor_SMD:C_0805_2012Metric_Pad1.18x1.45mm_HandSolder, F.Cu at (236.8, 186.9)
- added C113: 1uF, Capacitor_SMD:C_0805_2012Metric_Pad1.18x1.45mm_HandSolder, F.Cu at (241.5, 183.1)
- added C114: 1uF, Capacitor_SMD:C_0805_2012Metric_Pad1.18x1.45mm_HandSolder, F.Cu at (251.1, 183.0)
- added C401: 10pF, Capacitor_SMD:C_0603_1608Metric_Pad1.08x0.95mm_HandSolder, F.Cu at (171.8, 196.3)
- added C402: 10pF, Capacitor_SMD:C_0603_1608Metric_Pad1.08x0.95mm_HandSolder, F.Cu at (175.4, 190.1)
- added C403: 10pF, Capacitor_SMD:C_0603_1608Metric_Pad1.08x0.95mm_HandSolder, F.Cu at (178.8, 187.0)
- added C404: 10pF, Capacitor_SMD:C_0603_1608Metric_Pad1.08x0.95mm_HandSolder, F.Cu at (182.4, 183.3)
- added C601: 0.1uF, Capacitor_SMD:C_0603_1608Metric_Pad1.08x0.95mm_HandSolder, F.Cu at (170.7, 202.6)
- added C602: 0.1uF, Capacitor_SMD:C_0603_1608Metric_Pad1.08x0.95mm_HandSolder, F.Cu at (169.5, 215.5)
- added C8: 0.1uF, Capacitor_SMD:C_0805_2012Metric_Pad1.18x1.45mm_HandSolder, F.Cu at (176.0, 219.8)
- added C801: 0.1uF, Capacitor_SMD:C_0603_1608Metric_Pad1.08x0.95mm_HandSolder, F.Cu at (213.9, 212.4)
- added C805: 0.1uF, Capacitor_SMD:C_0603_1608Metric_Pad1.08x0.95mm_HandSolder, F.Cu at (207.0, 199.9)
- added C811: 0.1uF, Capacitor_SMD:C_0603_1608Metric_Pad1.08x0.95mm_HandSolder, F.Cu at (186.6, 201.1)
- added C812: 0.1uF, Capacitor_SMD:C_0603_1608Metric_Pad1.08x0.95mm_HandSolder, F.Cu at (196.1, 227.3)
- added C831: 10uF, Capacitor_SMD:C_0805_2012Metric_Pad1.18x1.45mm_HandSolder, F.Cu at (180.5, 212.0)
- added C862: 0.1uF, Capacitor_SMD:C_0603_1608Metric_Pad1.08x0.95mm_HandSolder, F.Cu at (186.9, 220.6)
- added D401: NM, Diode_SMD:D_SOD-123, F.Cu at (168.4, 193.5)
- added D402: NM, Diode_SMD:D_SOD-123, F.Cu at (172.1, 189.8)
- added D403: NM, Diode_SMD:D_SOD-123, F.Cu at (175.3, 186.7)
- added D404: NM, Diode_SMD:D_SOD-123, F.Cu at (179.0, 183.1)
- added J401: JTAG, Connector_PinHeader_2.54mm:PinHeader_2x05_P2.54mm_Vertical, F.Cu at (164.7, 182.9)
- added J601: Conn_01x07_Male, Connector_PinHeader_2.54mm:PinHeader_1x07_P2.54mm_Vertical, F.Cu at (162.2, 201.8)
- added Q2: MMBT3904, Package_TO_SOT_SMD:SOT-23_Handsoldering, F.Cu at (84.0, 225.0)
- added R101: 10K, Resistor_SMD:R_0805_2012Metric_Pad1.20x1.40mm_HandSolder, F.Cu at (252.0, 186.2)
- added R401: 10K, Resistor_SMD:R_0603_1608Metric_Pad0.98x0.95mm_HandSolder, F.Cu at (170.4, 192.0)
- added R402: 10K, Resistor_SMD:R_0603_1608Metric_Pad0.98x0.95mm_HandSolder, F.Cu at (172.7, 187.3)
- added R403: 10K, Resistor_SMD:R_0603_1608Metric_Pad0.98x0.95mm_HandSolder, F.Cu at (176.1, 184.3)
- added R404: 10K, Resistor_SMD:R_0603_1608Metric_Pad0.98x0.95mm_HandSolder, F.Cu at (179.7, 180.6)
- added R405: 1K, Resistor_SMD:R_0603_1608Metric_Pad0.98x0.95mm_HandSolder, F.Cu at (173.2, 194.8)
- added R5: 68R, Resistor_SMD:R_0805_2012Metric_Pad1.20x1.40mm_HandSolder, F.Cu at (174.5, 218.3)
- added R6: 75R, Resistor_SMD:R_0805_2012Metric_Pad1.20x1.40mm_HandSolder, F.Cu at (74.5, 225.0)
- added R601: 10K, Resistor_SMD:R_0805_2012Metric_Pad1.20x1.40mm_HandSolder, F.Cu at (168.1, 212.8)
- added R602: 10K, Resistor_SMD:R_0805_2012Metric_Pad1.20x1.40mm_HandSolder, F.Cu at (174.6, 201.8)
- added R7: 1K, Resistor_SMD:R_0805_2012Metric_Pad1.20x1.40mm_HandSolder, F.Cu at (84.5, 222.0)
- added R8: 10K, Resistor_SMD:R_0805_2012Metric_Pad1.20x1.40mm_HandSolder, F.Cu at (78.2, 224.0)
- added R801: 10K, Resistor_SMD:R_0603_1608Metric_Pad0.98x0.95mm_HandSolder, F.Cu at (178.0, 209.3)
- added R802: 10K, Resistor_SMD:R_0603_1608Metric_Pad0.98x0.95mm_HandSolder, F.Cu at (176.8, 208.1)
- added R803: 10K, Resistor_SMD:R_0603_1608Metric_Pad0.98x0.95mm_HandSolder, F.Cu at (203.5, 227.6)
- added R804: 10K, Resistor_SMD:R_0603_1608Metric_Pad0.98x0.95mm_HandSolder, F.Cu at (202.3, 228.8)
- added R805: 10K, Resistor_SMD:R_0603_1608Metric_Pad0.98x0.95mm_HandSolder, F.Cu at (201.2, 229.9)
- added R806: 10K, Resistor_SMD:R_0603_1608Metric_Pad0.98x0.95mm_HandSolder, F.Cu at (197.2, 228.4)
- added R807: 10K, Resistor_SMD:R_0603_1608Metric_Pad0.98x0.95mm_HandSolder, F.Cu at (181.7, 205.5)
- added R820: 22R, Resistor_SMD:R_0603_1608Metric_Pad0.98x0.95mm_HandSolder, F.Cu at (198.3, 231.1)
- added R831: 10K, Resistor_SMD:R_0603_1608Metric_Pad0.98x0.95mm_HandSolder, F.Cu at (179.2, 210.5)
- added U101: NCV8164ASN120T1G, Package_SO:TSOP-5_1.65x3.05mm_P0.95mm, F.Cu at (236.8, 184.1)
- added U102: BD33HC0WEFJ-E2, Package_SO:HTSOP-8-1EP_3.9x4.9mm_P1.27mm_EP2.4x3.2mm_ThermalVias, F.Cu at (246.3, 183.9)
- added U301: FSA2257MUX, Package_SO:MSOP-10_3x3mm_P0.5mm, F.Cu at (174.1, 101.6)
- added U601: W25Q128JVS, Package_SO:SOIC-8_5.23x5.23mm_P1.27mm, F.Cu at (171.2, 207.4)
- added U801: T8Q144, Package_QFP:TQFP-144_20x20mm_P0.5mm, F.Cu at (197.4, 210.9)
- C18: value 330uF/LOW_ESR -> 100uF; footprint Capacitor_SMD:CP_Elec_6.3x7.7 -> Capacitor_SMD:CP_Elec_6.3x5.3
- C19: value 10uF -> 0.1uF
- J14: value JTAG -> VSYNC_DISCRETE; footprint Connector_PinHeader_2.54mm:PinHeader_2x05_P2.54mm_Vertical -> BNC-THT:BNC-THT
- SW1, SW2: footprint PTS645:PTS645 -> Button_Switch_SMD:SW_SPST_EVQP7C
- U11: value BA33BC0FP-E2 -> 74LVC2G34; footprint Package_TO_SOT_SMD:TO-252-3_TabPin2 -> Package_TO_SOT_SMD:SOT-23-6_Handsoldering
- moved C18 178.9 mm to (75.8, 216.8)
- moved C19 178.2 mm to (80.8, 216.5)
- moved J14 117.6 mm to (59.4, 226.5), turned to 0 degrees
- moved D9 115.6 mm to (70.0, 222.4), turned to 270 degrees
- moved D10 111.1 mm to (70.0, 228.2), turned to 270 degrees
- moved U11 88.5 mm to (171.8, 222.6), turned to 45 degrees
- moved C59 60.0 mm to (193.6, 242.8), turned to 225 degrees
- moved C58 54.7 mm to (190.3, 239.2), turned to 225 degrees
- moved U9 34.3 mm to (196.2, 234.3), turned to 135 degrees
- moved C808 29.3 mm to (188.2, 221.9), turned to 225 degrees
- moved C851 29.3 mm to (209.2, 202.2), turned to 45 degrees
- moved C852 29.3 mm to (209.3, 219.6), turned to 315 degrees
- moved C855 28.9 mm to (201.9, 194.7), turned to 45 degrees
- moved C807 27.9 mm to (184.7, 218.4), turned to 225 degrees
- moved R88 27.2 mm to (190.2, 183.1), turned to 45 degrees
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- renumbered C31 to C802, C32 to C803, C33 to C804, C35 to C806, C36 to C807, C37 to C808, C38 to C809, C39 to C810, C60 to C851, C40 to C852, C41 to C853, C42 to C854, C43 to C855, C44 to C856, C45 to C857, C46 to C858, C47 to C859, C48 to C860, C49 to C861
Connections:
- C18 pad 1: +3V3 -> +5VA
- C19 pad 1: STBY_5V -> +5VA
- C802 pad 1: +3V3 -> +1V2
- C803 pad 1: +3V3 -> +1V2
- C804 pad 1: +3V3 -> +1V2
- C806 pad 1: +3V3 -> +1V2
- C807 pad 1: +3V3 -> +1V2
- C808 pad 1: +3V3 -> +1V2
- C809 pad 1: +3V3 -> +1V2
- C810 pad 1: +3V3 -> +1V2
- C9 pad 1: GND -> +5VA
- C9 pad 2: +5VA -> GND
- D10 pad 1: +3V3 -> Net-(D10-Pad1)
- D10 pad 2: /FPGA/TDO -> GND
- D9 pad 1: +3V3 -> +5VA
- D9 pad 2: /FPGA/TCK -> Net-(D10-Pad1)
- J14 pad 1: /FPGA/TCK -> Net-(D10-Pad1)
- SW1 pad 1: FORCE_VIDEO2 -> FORCE_VIDEO
- SW2 pad 1: FORCE_VIDEO -> FORCE_VIDEO2
- U11 pad 1: STBY_5V -> VSYNC_DISCRETE_IN
- U11 pad 3: +3V3 -> GND
Routing:
- net +1V2: track 0.00 -> 163.0 mm, vias 0 -> 13
- net VSYNC_DISCRETE_IN: track 0.00 -> 133.1 mm
- net +3V3: track 468.3 -> 546.9 mm, vias 23 -> 37
- net +5VA: track 593.0 -> 656.8 mm, vias 14 -> 17
- net NORM_Y_G: track 134.2 -> 90.4 mm
- net ~CRESET: track 0.00 -> 37.9 mm
- net ~VIDEO_OE: track 205.5 -> 171.3 mm, vias 5 -> 3
- net ~FPGA_CCK: track 0.00 -> 34.0 mm, vias 0 -> 1
- net ~FPGA_MISO: track 0.00 -> 30.6 mm, vias 0 -> 2
- net ~FPGA_SS: track 0.00 -> 30.6 mm
- net ~FPGA_MOSI: track 0.00 -> 30.3 mm, vias 0 -> 1
- net CDONE: track 0.00 -> 29.9 mm
- net /FPGA/TDI: track 25.3 -> 43.3 mm, vias 1 -> 2
- net GND: track 163.0 -> 145.0 mm, vias 63 -> 57
- net STBY_5V: track 69.1 -> 87.0 mm
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Other:
- board text added: "CCK"
- board text added: "CDONE"
- board text added: "HSYNC Max. 5Vpp"
- board text added: "MISO"
- board text added: "MOSI"
- board text added: "Rev. F1"
- board text added: "VSYNC IN Max. 5Vpp"
- board text added: "~CRESET"
- board text added: "~SS"
- board text removed: "Rev. E1"
