File: bkm-68x-simple.kicad_pcb (KiCad board)
At the start: 2 copper layers, 230.4 x 233.5 mm, 252 parts, among them CN985 mezz-conn-02x50, CN986 mezz-conn-02x50, J1 PR_R, J10 TP_VIDEO_OE, J11 TP_VSYNC, J12 JTAG, J13 PR_R_OUT, J14 VSYNC_DISCRETE, J15 Y_G_OUT, J16 PB_B_OUT, J17 EXT_SYNC_OUT, J18 Conn_01x02_Male, J19 TP_NORM_Y_G, J2 Y_G, J20 TP_RGB_COMP_X, J21 TP_HD_SD_X, J22 VSYNC_DISCRETE_OUT, J3 PB_B, J4 EXT_SYNC, J401 JTAG, J5 TP_Y_G, J6 TP_PB_B, J601 Conn_01x07_Male, J7 TP_PR_R, J8 TP_HSYNC, J9 TP_INT_EXT_SYNC, Q1 MMBT3904, Q2 MMBT3904, SW1 FORCE_VIDEO, SW2 FORCE_VIDEO, SW3 PR_R_TERM, SW4 Y_G_TERM, SW5 PB_B_TERM, SW6 EXT_SYNC_TERM, SW7 EXT_SYNC_TERM, U1 ADG1611BCPZ, U10 74LVC541A, U101 NCV8164ASN120T1G, U102 BD33HC0WEFJ-E2, U11 74LVC2G34, U12 TC7SZ125FU, U13 LM2990SX-5.0, U14 BA50BC0FP-E2, U16 SN74LVC1G14DBV, U17 ISL4089, U19 74LVC2G34, U2 THS7374, U3 ISL59885, U301 FSA2257MUX, U5 74LVC14A, U6 74LVC14A, U601 W25Q128JVS, U7 74LVC14A, U8 TC7WH125, U801 T8Q144, U9 KC2520Z50

Commit message: Rev. F2
Parts:
- added J101: TP_1V2, TestPoint:TestPoint_Pad_D2.0mm, F.Cu at (232.7, 188.3)
- added J102: TP_3V3, TestPoint:TestPoint_Pad_D2.0mm, F.Cu at (229.4, 181.9)
- added J103: TP_GNDD1, TestPoint:TestPoint_Pad_D2.0mm, F.Cu at (229.5, 172.3)
- added J201: TP_NEG5V, TestPoint:TestPoint_Pad_D2.0mm, F.Cu at (264.9, 103.3)
- added J202: TP_5V, TestPoint:TestPoint_Pad_D2.0mm, F.Cu at (236.0, 119.4)
- added J203: TP_GNDA1, TestPoint:TestPoint_Pad_D2.0mm, F.Cu at (217.8, 97.7)
Routing:
- net -5VA: track 47.8 -> 56.5 mm
- net +3V3: track 546.9 -> 547.0 mm, vias 37 -> 38
- net +5VA: vias 17 -> 18
- net +1V2: vias 13 -> 14
Other:
- board text added: "Rev. F2"
- board text added: "TP_1V2"
- board text added: "TP_3V3"
- board text added: "TP_5V"
- board text added: "TP_GND"
- board text added: "TP_NEG5V"
- board text removed: "Rev. F1"

Commit message: Rev. F4
Parts:
- added C30: NM, Capacitor_SMD:C_0805_2012Metric_Pad1.18x1.45mm_HandSolder, F.Cu at (234.2, 73.6)
- added C31: NM, Capacitor_SMD:C_0805_2012Metric_Pad1.18x1.45mm_HandSolder, F.Cu at (234.2, 76.9)
- added C32: NM, Capacitor_SMD:C_0805_2012Metric_Pad1.18x1.45mm_HandSolder, F.Cu at (234.2, 80.3)
- added C33: 22pF, Capacitor_SMD:C_0805_2012Metric_Pad1.18x1.45mm_HandSolder, F.Cu at (187.7, 97.7)
- added R44: 1K, Resistor_SMD:R_0805_2012Metric_Pad1.20x1.40mm_HandSolder, F.Cu at (194.1, 101.2)
- added U501: ADG1611, Package_SO:TSSOP-16_4.4x5mm_P0.65mm, F.Cu at (254.3, 76.5)
- J601: value Conn_01x07_Male -> SPI_PROG
- moved J7 2.47 mm to (264.3, 73.9)
- moved R10 2.23 mm to (243.0, 73.6)
- moved R9 2.23 mm to (238.1, 73.6)
- moved R11 2.22 mm to (238.1, 76.9)
- moved R12 2.22 mm to (243.0, 76.9)
- moved R13 2.22 mm to (238.1, 80.3)
- moved R14 2.22 mm to (243.0, 80.3)
- moved C62 2.00 mm to (190.6, 105.6)
- moved C65 2.00 mm to (194.2, 109.5)
- moved R84 2.00 mm to (194.1, 107.4)
- moved U16 2.00 mm to (193.4, 104.3)
- moved C1 1.78 mm to (248.5, 79.7)
- moved C2 1.52 mm to (259.9, 74.8)
Connections:
- net Net-(R10-Pad2) renamed /Video/PR_R_L
- net Net-(R11-Pad2) renamed /Video/Y_G_L
- net Net-(R13-Pad2) renamed /Video/PB_B_L
- U16 pad 4: /Video/~CSYNC -> Net-(R44-Pad2)
Routing:
- net ~VIDEO_OE: track 171.3 -> 181.2 mm, vias 3 -> 4
- net +5VA: track 652.7 -> 658.3 mm
- net GND: track 145.0 -> 150.6 mm, vias 57 -> 54
- net /Video/PR_R_L: track 14.6 -> 18.3 mm
- net Net-(R44-Pad2): track 0.00 -> 2.78 mm
- net /Video/Y_G_L: track 12.6 -> 15.4 mm
- net /Video/PB_B_L: track 14.3 -> 17.0 mm
- net PR_R_AMP: track 89.7 -> 87.3 mm
- net PB_B_AMP: track 87.5 -> 85.2 mm
- net Y_G: track 25.5 -> 27.8 mm
- net Y_G_SW: track 79.0 -> 76.9 mm
- net -5VA: track 56.5 -> 58.6 mm
- net PB_B: track 21.9 -> 23.9 mm
Other:
- board text added: "Rev. F4"
- board text removed: "Rev. F2"
