File: fpga.sch (KiCad schematic (older format))
At the start: 107 parts, among them J14 JTAG, J19 TP_NORM_Y_G, J20 TP_RGB_COMP_X, J21 TP_HD_SD_X, SW1 FORCE_VIDEO, SW2 FORCE_VIDEO, U10 74LVC541A, U12 TC7SZ125FU, U15 10M08SC, U19 74LVC2G34, U5 74LVC14A, U6 74LVC14A, U7 74LVC14A, U9 KC2520Z50

Commit message: Rev. F1
Parts:
- removed R44, R45, R73: 10K, Resistor_SMD:R_0805_2012Metric_Pad1.20x1.40mm_HandSolder, symbol bkm-68x-simple-rescue:R
- removed U15: 10M08SC, Package_QFP:EQFP-144-1EP_20x20mm_P0.5mm_EP8.93x8.7mm_ThermalVias, symbol bkm-68x-simple-rescue:10M08SC-FPGA_Intel
- added C601, C602, C862: 0.1uF, Capacitor_SMD:C_0603_1608Metric_Pad1.08x0.95mm_HandSolder, symbol Device:C
- added C8: 0.1uF, Capacitor_SMD:C_0805_2012Metric_Pad1.18x1.45mm_HandSolder, symbol Device:C
- added C831: 10uF, Capacitor_SMD:C_0805_2012Metric_Pad1.18x1.45mm_HandSolder, symbol Device:C
- added J601: Conn_01x07_Male, Connector_PinHeader_2.54mm:PinHeader_1x07_P2.54mm_Vertical, symbol Connector:Conn_01x07_Male
- added R401, R402, R801, R802, R803, R804, R805, R806, R807, R831: 10K, Resistor_SMD:R_0603_1608Metric_Pad0.98x0.95mm_HandSolder, symbol bkm-68x-simple-rescue:R
- added R5: 68R, Resistor_SMD:R_0805_2012Metric_Pad1.20x1.40mm_HandSolder, symbol bkm-68x-simple-rescue:R
- added R601, R602: 10K, Resistor_SMD:R_0805_2012Metric_Pad1.20x1.40mm_HandSolder, symbol bkm-68x-simple-rescue:R
- added R820: 22R, Resistor_SMD:R_0603_1608Metric_Pad0.98x0.95mm_HandSolder, symbol bkm-68x-simple-rescue:R
- added U11: 74LVC2G34, Package_TO_SOT_SMD:SOT-23-6_Handsoldering, symbol 74LVCxG34:74LVC2G34
- added U601: W25Q128JVS, Package_SO:SOIC-8_5.23x5.23mm_P1.27mm, symbol Memory_Flash:W25Q128JVS
- added U801: T8Q144, Package_QFP:TQFP-144_20x20mm_P0.5mm, symbol bkm-68x-simple-rescue:T8Q144-Efinix_FPGA
- R403: renamed from R75; footprint Resistor_SMD:R_0805_2012Metric_Pad1.20x1.40mm_HandSolder -> Resistor_SMD:R_0603_1608Metric_Pad0.98x0.95mm_HandSolder
- R404: renamed from R74; footprint Resistor_SMD:R_0805_2012Metric_Pad1.20x1.40mm_HandSolder -> Resistor_SMD:R_0603_1608Metric_Pad0.98x0.95mm_HandSolder
- R405: renamed from R76; footprint Resistor_SMD:R_0805_2012Metric_Pad1.20x1.40mm_HandSolder -> Resistor_SMD:R_0603_1608Metric_Pad0.98x0.95mm_HandSolder
- SW1, SW2: footprint PTS645:PTS645 -> Button_Switch_SMD:SW_SPST_EVQP7C
- renumbered C50 to C401, C51 to C402, C52 to C403, C53 to C404, C60 to C851, C40 to C852, C41 to C853, C42 to C854, C43 to C855, C44 to C856, C45 to C857, C46 to C858, C47 to C859, C48 to C860, C49 to C861, D9 to D401, D10 to D402, D11 to D403, D12 to D404, J14 to J401
Connections:
- net +3V3: now also C601.2, C602.1, C8.2, C862.1, R401.2, R402.2, R601.2, R602.2, R801.1, R802.1, R803.1, R804.1, R805.1, R806.1, R807.2, R831.2, U11.5 (VCC), U601.8 (VCC), U801.12 (VCCIO1C_1D), U801.122 (VCCIO_3A), U801.143 (VCCIO_1E), U801.21 (VCCIO_1B), U801.23 (VCCIO_1A), U801.51 (VCCIO4B), U801.52 (VCCIO4B), U801.62 (VCCIO4A), U801.63 (VCCIO4A), U801.88 (VCCIO3E), U801.91 (VCCIO3D), U801.95 (VCCIO3B_3C)
- net CLK_50MHz: now also R820.1
- net DBG1: now also U801.71 (GPIOB_CLKP0)
- net DBG2: now also U801.72 (GPIOB_CLKN0)
- net FORCE_VIDEO: now also SW1.1 (A), U801.40 (GPIOB_TXP02); no longer SW2.1 (A)
- net FORCE_VIDEO2: now also SW2.1 (A), U801.42 (GPIOB_TXP04); no longer SW1.1 (A)
- net FPGA_ADIN0: now also U801.105 (GPIOR_95_CDI26)
- net FPGA_ADIN1: now also U801.101 (GPIOR_112_CDI23)
- net FPGA_ADIN2: now also U801.100 (GPIOR_113_CDI22)
- net FPGA_ADIN3: now also U801.106 (GPIOR_94_CDI27)
- net FPGA_ADIN4: now also U801.99 (GPIOR_116_CTRL15)
- net FPGA_ADIN5: now also U801.98 (GPIOR_117_CTRL14)
- net FPGA_ADIN6: now also U801.97 (GPIOR_122_CLK13_CDI21)
- net FPGA_ADIN7: now also U801.93 (GPIOR_123_CLK12_CDI20)
- net FPGA_ADOUT0: now also U801.118 (GPIOR_79_EXTFB1_CDI30)
- net FPGA_ADOUT1: now also U801.117 (GPIOR_80)
- net FPGA_ADOUT2: now also U801.116 (GPIOR_81_MREFCLK)
- net FPGA_ADOUT3: now also U801.115 (GPIOR_82)
- net FPGA_ADOUT4: now also U801.114 (GPIOR_83)
- net FPGA_ADOUT5: now also U801.113 (GPIOR_84)
- net FPGA_ADOUT6: now also U801.112 (GPIOR_86)
- net FPGA_ADOUT7: now also U801.111 (GPIOR_85)
- net FPGA_CLK_RW: now also U801.83 (GPIOR_136_CDI16)
- net FPGA_R_~W: now also U801.86 (GPIOR133_CDI18)
- net FPGA_~A~_D: now also U801.87 (GPIOR_132_CDI19)
- net GND: now also C601.1, C602.2, C8.1, C831.2, C862.2, J601.7 (Pin_7), U11.2 (GND), U11.3 (1A), U601.4 (GND)
- net HD_SD_X: now also U801.61 (GPIOB_RXP03)
- net HSYNC_SEP_BUF: now also U801.3 (GPIOL_53_CDI10)
- net RGB_COMP_X: now also U801.66 (GPIOB_RXP07)
- net TCK: now also R401.1, U801.26 (TCK)
- net TDI: now also U801.27 (TDI)
- net TDO: now also R402.1, U801.24 (TDO)
- net TMS: now also U801.25 (TMS)
- net VSYNC_SEP_BUF: now also U801.4 (GPIOL_54_CDI11)
- net ~FPGA_AD_OE: now also U801.119 (GPIOR_78_EXTFB0_CDI31)
- net ~FPGA_IRQ: now also U801.81 (GPIOR_139)
- net ~FPGA_IRQ_OE: now also U801.82 (GPIOR_138)
- net ~FPGA_RESET: now also U801.109 (GPIOR_88_CDI28)
- net ~FPGA_SLOT: now also U801.84 (GPIOR_135_CDI17)
- net ~VIDEO_OE: now also U801.140 (GPIOL_67_CDI13)
- net at R79.1: now also U801.135 (GPIOL_72_EXTFB0_CDI14)
- net at R78.1: now also U801.134 (GPIOL_73_EXTFB1_CDI15)
- net at R87.1: now also U801.6 (GPIOL_46)
- net at R88.1: now also U801.7 (GPIOL_41_CDI9)
- new net: R601.1, U601.3 (IO2)
- new net: R602.1, U601.7 (IO3)
- new net: R5.2, U11.6 (1Y)
- new net: R802.2, U801.32 (GPIOL_04_CSI)
- new net: R803.2, U801.80 (GPIOR_149_CBUS2)
- new net: R804.2, U801.79 (GPIOR_150_CBUS1)
- new net: R805.2, U801.78 (GPIOR_151_CBUS0)
- new net: R806.2, U801.74 (GPIOR_158_TEST_N)
- new net: R820.2, U801.75 (GPIOR_157_PLLIN)
- new net CDONE: J601.6 (Pin_6), R801.2, U801.34 (CDONE)
- new net VSYNC_DISCRETE_BUF: R5.1, U801.38 (GPIOB_TXP00)
- new net VSYNC_DISCRETE_IN: U11.1 (1A)
- new net ~CRESET: C831.1, J601.5 (Pin_5), R831.1, U801.35 (CRESET_N)
- new net ~FPGA_CCK: J601.1 (Pin_1), U601.6 (CLK), U801.30 (GPIOL_01_CCK)
- new net ~FPGA_MISO: J601.3 (Pin_3), U601.2 (DO(IO1)), U801.28 (GPIOL_09_CDI1)
- new net ~FPGA_MOSI: J601.4 (Pin_4), U601.5 (DI(IO0)), U801.29 (GPIOL_08_CDI0)
- new net ~FPGA_SS: J601.2 (Pin_2), R807.1, U601.1 (~CS), U801.31 (GPIOL_00_SS_N)
- no-connect marks 64 -> 9
Other:
- moved on the sheet: C401, C402, C403, C404, C71, D13, D14, D401, D402, D403, D404, J401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

Commit message: Rev. F2
Parts:
- C12, C20, C21, C22, C71, C8: JLC (none) -> 0805; LCSC (none) -> C77082
- C401, C402, C403, C404: JLC (none) -> 0603; LCSC (none) -> C106245
- C601, C602, C851, C852, C853, C854, C855, C856, C857, C858, C859, C860, C861, C862: JLC (none) -> 0603; LCSC (none) -> C85864
- C831: JLC (none) -> 0805; LCSC (none) -> C126586
- R15, R16, R17, R18, R19, R20, R21, R22, R23, R25, R36, R38, R42, R43, R47, R48, R49, R5, R50, R51, R52, R53, R62, R63, R64, R65, R66, R67: JLC (none) -> 0805; LCSC (none) -> C137498
- R24, R26, R27, R28, R29, R30, R31, R32: JLC (none) -> 0805; LCSC (none) -> C114541
- R33, R34, R35, R39: JLC (none) -> 0805; LCSC (none) -> C126351
- R37: JLC (none) -> 0805; LCSC (none) -> C114565
- R40, R41, R54, R55, R56, R57, R58, R59, R60, R61, R68, R69, R70, R78, R79, R87, R88: JLC (none) -> 0805; LCSC (none) -> C107702
- R401, R402, R403, R404, R801, R802, R803, R804, R805, R806, R807, R831: JLC (none) -> 0603; LCSC (none) -> C98220
- R405: JLC (none) -> 0603; LCSC (none) -> C22548
- R46, R601, R602, R77: JLC (none) -> 0805; LCSC (none) -> C84376
- R82: JLC (none) -> 0805; LCSC (none) -> C114564
- R820: JLC (none) -> 0603; LCSC (none) -> C107701
- R83: JLC (none) -> 0805; LCSC (none) -> C114543
- U10: JLC (none) -> TSSOP-14; LCSC (none) -> C34495
- U11, U19: JLC (none) -> SOT-23-6; LCSC (none) -> C347589
- U12: JLC (none) -> SC-70-5; LCSC (none) -> C7833
- U5, U6, U7: JLC (none) -> TSSOP-14; LCSC (none) -> C6066
- U601: JLC (none) -> SOIC-8_208mil; LCSC (none) -> C97521
- U9: JLC (none) -> SMD2520-4P; LCSC (none) -> C2916926
