File: fpga.sch (KiCad schematic (older format))
At the start: 126 parts, among them J19 TP_NORM_Y_G, J20 TP_RGB_COMP_X, J21 TP_HD_SD_X, J401 JTAG, J601 Conn_01x07_Male, SW1 FORCE_VIDEO, SW2 FORCE_VIDEO, U10 74LVC541A, U11 74LVC2G34, U12 TC7SZ125FU, U19 74LVC2G34, U5 74LVC14A, U6 74LVC14A, U601 W25Q128JVS, U7 74LVC14A, U801 T8Q144, U9 KC2520Z50

Commit message: Rev. F4
Parts:
- J601: value Conn_01x07_Male -> SPI_PROG
Changed lines of the file:
@@
 P 12600 7050
 F 0 "J601" H 12708 7531 50  0000 C CNN
-F 1 "Conn_01x07_Male" H 12708 7440 50  0000 C CNN
+F 1 "SPI_PROG" H 12708 7440 50  0000 C CNN
 F 2 "Connector_PinHeader_2.54mm:PinHeader_1x07_P2.54mm_Vertical" H 12600 7050 50  0001 C CNN
 F 3 "~" H 12600 7050 50  0001 C CNN
