File: power-supply.sch (KiCad schematic (older format))
At the start: 42 parts, among them J18 Conn_01x02_Male, U101 NCV8164ASN120T1G, U102 BD33HC0WEFJ-E2, U13 LM2990SX-5.0, U14 BA50BC0FP-E2, U801 T8Q144

Commit message: Rev. F2
Parts:
- added J101: TP_1V2, TestPoint:TestPoint_Pad_D2.0mm, symbol bkm-68x-simple-rescue:TEST_1P
- added J102: TP_3V3, TestPoint:TestPoint_Pad_D2.0mm, symbol bkm-68x-simple-rescue:TEST_1P
- added J103: TP_GNDD1, TestPoint:TestPoint_Pad_D2.0mm, symbol bkm-68x-simple-rescue:TEST_1P
- added J201: TP_NEG5V, TestPoint:TestPoint_Pad_D2.0mm, symbol bkm-68x-simple-rescue:TEST_1P
- added J202: TP_5V, TestPoint:TestPoint_Pad_D2.0mm, symbol bkm-68x-simple-rescue:TEST_1P
- added J203: TP_GNDA1, TestPoint:TestPoint_Pad_D2.0mm, symbol bkm-68x-simple-rescue:TEST_1P
- C111, C112, C113, C114, C23: JLC (none) -> 0805; LCSC (none) -> C28323
- C14, C16, C18, C24, C58, C61: JLC (none) -> SMD,6.3x5.5mm; LCSC (none) -> C111600
- C15, C17, C19, C56, C57, C59: JLC (none) -> 0805; LCSC (none) -> C77082
- C25, C28, C68, C70: JLC (none) -> 0805; LCSC (none) -> C126586
- C26, C29: JLC (none) -> SMD,6.3x5.4mm; LCSC (none) -> C413670
- C801, C802, C803, C804, C805, C806, C807, C808, C809, C810, C811, C812: JLC (none) -> 0603; LCSC (none) -> C85864
- R101: JLC (none) -> 0805; LCSC (none) -> C84376
- U101: JLC (none) -> TSOP-5; LCSC (none) -> C2902277
- U13: JLC (none) -> TO-263-3; LCSC (none) -> C201697
- U14: JLC (none) -> TO-252-3; LCSC (none) -> C2909275
Connections:
- net +1V2: now also J101.1
- net +3V3: now also J102.1
- net +5VA: now also J202.1
- net -5VA: now also J201.1
- net GNDA: now also J203.1
- net GNDD: now also J103.1
